Commit message: Joints: BrainCo hands in the 3D model, fingers drawn from the robot's readings

File: public/g1/g1.urdf (robot description, URDF)
Before this commit: robot g1_29dof_rev_1_0_with_inspire_hand_DFQ, 63 links, 62 joints
Links:
- removed link L_hand_base_link
- removed link L_index_intermediate
- removed link L_index_proximal
- removed link L_middle_intermediate
- removed link L_middle_proximal
- removed link L_pinky_intermediate
- removed link L_pinky_proximal
- removed link L_ring_intermediate
- removed link L_ring_proximal
- removed link L_thumb_distal
- removed link L_thumb_intermediate
- removed link L_thumb_proximal
- removed link L_thumb_proximal_base
- removed link R_hand_base_link
- removed link R_index_intermediate
- removed link R_index_proximal
- removed link R_middle_intermediate
- removed link R_middle_proximal
- removed link R_pinky_intermediate
- removed link R_pinky_proximal
- removed link R_ring_intermediate
- removed link R_ring_proximal
- removed link R_thumb_distal
- removed link R_thumb_intermediate
- removed link R_thumb_proximal
- removed link R_thumb_proximal_base
- removed link pelvis_contour_link
- added link left_base2_link, mass 0.02280635; visual mesh filename=meshes/left_base2_link.STL
- added link left_base_link, mass 0.238; visual mesh filename=meshes/left_base_link.STL
- added link left_index_distal_Link, mass 0.009; visual mesh filename=meshes/left_index_distal_Link.STL
- added link left_index_proximal_Link, mass 0.009; visual mesh filename=meshes/left_index_proximal_Link.STL
- added link left_index_tip_Link, mass 0.001; visual mesh filename=meshes/left_index_tip_Link.STL
- added link left_middle_distal_Link, mass 0.009; visual mesh filename=meshes/left_middle_distal_Link.STL
- added link left_middle_proximal_Link, mass 0.009; visual mesh filename=meshes/left_middle_proximal_Link.STL
- added link left_middle_tip_Link, mass 0.001; visual mesh filename=meshes/left_middle_tip_Link.STL
- added link left_pinky_distal_Link, mass 0.009; visual mesh filename=meshes/left_pinky_distal_Link.STL
- added link left_pinky_proximal_Link, mass 0.009; visual mesh filename=meshes/left_pinky_proximal_Link.STL
- added link left_pinky_tip_Link, mass 0.001; visual mesh filename=meshes/left_pinky_tip_Link.STL
- added link left_ring_distal_Link, mass 0.009; visual mesh filename=meshes/left_ring_distal_Link.STL
- added link left_ring_proximal_Link, mass 0.009; visual mesh filename=meshes/left_ring_proximal_Link.STL
- added link left_ring_tip_Link, mass 0.001; visual mesh filename=meshes/left_ring_tip_Link.STL
- added link left_thumb_distal_Link, mass 0.01; visual mesh filename=meshes/left_thumb_distal_Link.STL
- added link left_thumb_metacarpal_Link, mass 0.01; visual mesh filename=meshes/left_thumb_metacarpal_Link.STL
- added link left_thumb_proximal_Link, mass 0.05; visual mesh filename=meshes/left_thumb_proximal_Link.STL
- added link left_thumb_tip_Link, mass 0.001; visual mesh filename=meshes/left_thumb_tip_Link.STL
- added link right_base2_link, mass 0.02280635; visual mesh filename=meshes/right_base2_link.STL
- added link right_base_link, mass 0.238; visual mesh filename=meshes/right_base_link.STL
- added link right_index_distal_link, mass 0.009; visual mesh filename=meshes/right_index_distal_link.STL
- added link right_index_proximal_link, mass 0.009; visual mesh filename=meshes/right_index_proximal_link.STL
- added link right_index_tip, mass 0.001; visual mesh filename=meshes/right_index_tip.STL
- added link right_middle_distal_link, mass 0.009; visual mesh filename=meshes/right_middle_distal_link.STL
- added link right_middle_proximal_link, mass 0.009; visual mesh filename=meshes/right_middle_proximal_link.STL
- added link right_middle_tip, mass 0.001; visual mesh filename=meshes/right_middle_tip.STL
- added link right_pinky_distal_link, mass 0.009; visual mesh filename=meshes/right_pinky_distal_link.STL
- added link right_pinky_proximal_link, mass 0.009; visual mesh filename=meshes/right_pinky_proximal_link.STL
- added link right_pinky_tip, mass 0.001; visual mesh filename=meshes/right_pinky_tip.STL
- added link right_ring_distal_link, mass 0.009; visual mesh filename=meshes/right_ring_distal_link.STL
- added link right_ring_proximal_link, mass 0.009; visual mesh filename=meshes/right_ring_proximal_link.STL
- added link right_ring_tip, mass 0.001; visual mesh filename=meshes/right_ring_tip.STL
- added link right_thumb_distal_link, mass 0.01; visual mesh filename=meshes/right_thumb_distal_link.STL
- added link right_thumb_metacarpal_link, mass 0.01; visual mesh filename=meshes/right_thumb_metacarpal_link.STL
- added link right_thumb_proximal_link, mass 0.05; visual mesh filename=meshes/right_thumb_proximal_link.STL
- added link right_thumb_tip, mass 0.001; visual mesh filename=meshes/right_thumb_tip.STL
- link pelvis: geometry visual mesh filename=meshes/pelvis_ver0529.STL
Joints:
- removed joint L_base_link_joint
- removed joint L_index_intermediate_joint
- removed joint L_index_proximal_joint
- removed joint L_middle_intermediate_joint
- removed joint L_middle_proximal_joint
- removed joint L_pinky_intermediate_joint
- removed joint L_pinky_proximal_joint
- removed joint L_ring_intermediate_joint
- removed joint L_ring_proximal_joint
- removed joint L_thumb_distal_joint
- removed joint L_thumb_intermediate_joint
- removed joint L_thumb_proximal_pitch_joint
- removed joint L_thumb_proximal_yaw_joint
- removed joint R_base_link_joint
- removed joint R_index_intermediate_joint
- removed joint R_index_proximal_joint
- removed joint R_middle_intermediate_joint
- removed joint R_middle_proximal_joint
- removed joint R_pinky_intermediate_joint
- removed joint R_pinky_proximal_joint
- removed joint R_ring_intermediate_joint
- removed joint R_ring_proximal_joint
- removed joint R_thumb_distal_joint
- removed joint R_thumb_intermediate_joint
- removed joint R_thumb_proximal_pitch_joint
- removed joint R_thumb_proximal_yaw_joint
- removed joint pelvis_contour_joint
- added joint left_base2_joint: type fixed, parent left_wrist_yaw_link, child left_base2_link, origin xyz=0.0415 0 0 rpy=0 0 0
- added joint left_base_joint: type fixed, parent left_wrist_yaw_link, child left_base_link, origin xyz=0.0591 0 0 rpy=-1.570796326 0 -1.570796326
- added joint left_index_distal_joint: type revolute, parent left_index_proximal_Link, child left_index_distal_Link, origin xyz=0 0 0.032 rpy=0 0 0, axis 0 1 0, limit lower=0 upper=1.693 effort=2 velocity=2.2685, mimic joint=left_index_proximal_joint multiplier=1.155 offset=0
- added joint left_index_proximal_joint: type revolute, parent left_base_link, child left_index_proximal_Link, origin xyz=-0.0021349 -0.029578 0.080876 rpy=0.11819 0.14743 0.17422, axis 0 1 0, limit lower=0 upper=1.4661 effort=2 velocity=2.2685
- added joint left_index_tip_joint: type fixed, parent left_index_distal_Link, child left_index_tip_Link, origin xyz=0.011097 0 0.035739 rpy=0 1.48723 0
- added joint left_middle_distal_joint: type revolute, parent left_middle_proximal_Link, child left_middle_distal_Link, origin xyz=0 0 0.037 rpy=0 0.12654 0, axis 0 1 0, limit lower=0 upper=1.693 effort=2 velocity=2.2685, mimic joint=left_middle_proximal_joint multiplier=1.155 offset=0
- added joint left_middle_proximal_joint: type revolute, parent left_base_link, child left_middle_proximal_Link, origin xyz=-0.0045935 -0.010061 0.084993 rpy=0.039468 0.1483 0.057975, axis 0 1 0, limit lower=0 upper=1.4661 effort=2 velocity=2.2685
- added joint left_middle_tip_joint: type fixed, parent left_middle_distal_Link, child left_middle_tip_Link, origin xyz=0.0073534 0 0.041703 rpy=0 1.34907 0
- added joint left_pinky_distal_joint: type revolute, parent left_pinky_proximal_Link, child left_pinky_distal_Link, origin xyz=0 0 0.029 rpy=0 0 0, axis 0 1 0, limit lower=0 upper=1.693 effort=2 velocity=2.2685, mimic joint=left_pinky_proximal_joint multiplier=1.155 offset=0
- added joint left_pinky_proximal_joint: type revolute, parent left_base_link, child left_pinky_proximal_Link, origin xyz=-0.0023733 0.029356 0.078694 rpy=-0.11815 0.14491 -0.17392, axis 0 1 0, limit lower=0 upper=1.4661 effort=2 velocity=2.2685
- added joint left_pinky_tip_joint: type fixed, parent left_pinky_distal_Link, child left_pinky_tip_Link, origin xyz=0.010221 0 0.032918 rpy=0 1.4756 0
- added joint left_ring_distal_joint: type revolute, parent left_ring_proximal_Link, child left_ring_distal_Link, origin xyz=0 0 0.035 rpy=0 0.12654 0, axis 0 1 0, limit lower=0 upper=1.693 effort=2 velocity=2.2685, mimic joint=left_ring_proximal_joint multiplier=1.155 offset=0
- added joint left_ring_proximal_joint: type revolute, parent left_base_link, child left_ring_proximal_Link, origin xyz=-0.00468767815858587 0.0100262714211602 0.0839819548795939 rpy=-0.0394618478609065 0.147209177132223 -0.0579317909005277, axis 0 1 0, limit lower=0 upper=1.4661 effort=2 velocity=2.2685
- added joint left_ring_tip_joint: type fixed, parent left_ring_distal_Link, child left_ring_tip_Link, origin xyz=0.0071824 0 0.040734 rpy=0 1.34907 0
- added joint left_thumb_distal_joint: type revolute, parent left_thumb_proximal_Link, child left_thumb_distal_Link, origin xyz=0 0.052 0 rpy=0 0 0, axis 1 0 0, limit lower=0 upper=1.0472 effort=1.1 velocity=2.5303, mimic joint=left_thumb_proximal_joint multiplier=1 offset=0
- added joint left_thumb_metacarpal_joint: type revolute, parent left_base_link, child left_thumb_metacarpal_Link, origin xyz=0.0045 -0.019 0.027825 rpy=0 0 0.16787, axis 0 0 1, limit lower=0 upper=1.5184 effort=0.5 velocity=2.6175
- added joint left_thumb_proximal_joint: type revolute, parent left_thumb_metacarpal_Link, child left_thumb_proximal_Link, origin xyz=0 -0.014227 0 rpy=0.17488 -0.23736 2.9737, axis 1 0 0, limit lower=0 upper=1.0472 effort=1.1 velocity=2.5303
- added joint left_thumb_tip_joint: type fixed, parent left_thumb_distal_Link, child left_thumb_tip_Link, origin xyz=0 0.026528781163583 -0.00177344281307927 rpy=0.0667504507 -0 3.14159265
- added joint right_base2_joint: type fixed, parent right_wrist_yaw_link, child right_base2_link, origin xyz=0.0415 0 0 rpy=0 0 0
- added joint right_base_joint: type fixed, parent right_wrist_yaw_link, child right_base_link, origin xyz=0.0591 0 0 rpy=1.570796326 0 1.570796326
- added joint right_index_distal_joint: type revolute, parent right_index_proximal_link, child right_index_distal_link, origin xyz=0 0 0.032 rpy=0 0 0, axis 0 1 0, limit lower=0 upper=1.693 effort=2 velocity=2.2685, mimic joint=right_index_proximal_joint multiplier=1.155 offset=0
- added joint right_index_proximal_joint: type revolute, parent right_base_link, child right_index_proximal_link, origin xyz=-0.0021181 0.029568 0.080876 rpy=-0.11819 0.14743 -0.17422, axis 0 1 0, limit lower=0 upper=1.4661 effort=2 velocity=2.2685
- added joint right_index_tip_joint: type fixed, parent right_index_distal_link, child right_index_tip, origin xyz=0.011097 0 0.035739 rpy=0 0.4756 0
- added joint right_middle_distal_joint: type revolute, parent right_middle_proximal_link, child right_middle_distal_link, origin xyz=0 0 0.037 rpy=0 0 0, axis 0 1 0, limit lower=0 upper=1.693 effort=2 velocity=2.2685, mimic joint=right_middle_proximal_joint multiplier=1.155 offset=0
- added joint right_middle_proximal_joint: type revolute, parent right_base_link, child right_middle_proximal_link, origin xyz=-0.0045767 0.010051 0.084993 rpy=-0.039468 0.1483 -0.057975, axis 0 1 0, limit lower=0 upper=1.4661 effort=2 velocity=2.2685
- added joint right_middle_tip_joint: type fixed, parent right_middle_distal_link, child right_middle_tip, origin xyz=0.012558 0 0.040442 rpy=0 0.4756 0
- added joint right_pinky_distal_joint: type revolute, parent right_pinky_proximal_link, child right_pinky_distal_link, origin xyz=0 0 0.029 rpy=0 0 0, axis 0 1 0, limit lower=0 upper=1.693 effort=2 velocity=2.2685, mimic joint=right_pinky_proximal_joint multiplier=1.155 offset=0
- added joint right_pinky_proximal_joint: type revolute, parent right_base_link, child right_pinky_proximal_link, origin xyz=-0.0023566 -0.029366 0.078694 rpy=0.11815 0.14491 0.17392, axis 0 1 0, limit lower=0 upper=1.4661 effort=2 velocity=2.2685
- added joint right_pinky_tip_joint: type fixed, parent right_pinky_distal_link, child right_pinky_tip, origin xyz=0.010221 0 0.032918 rpy=0 0.4756 0
- added joint right_ring_distal_joint: type revolute, parent right_ring_proximal_link, child right_ring_distal_link, origin xyz=0 0 0.035 rpy=0 0 0, axis 0 1 0, limit lower=0 upper=1.693 effort=2 velocity=2.2685, mimic joint=right_ring_proximal_joint multiplier=1.155 offset=0
- added joint right_ring_proximal_joint: type revolute, parent right_base_link, child right_ring_proximal_link, origin xyz=-0.0046709 -0.010037 0.083982 rpy=0.039462 0.14721 0.057932, axis 0 1 0, limit lower=0 upper=1.4661 effort=2 velocity=2.2685
- added joint right_ring_tip_joint: type fixed, parent right_ring_distal_link, child right_ring_tip, origin xyz=0.012266 0 0.039501 rpy=0 0.4756 0
- added joint right_thumb_distal_joint: type revolute, parent right_thumb_proximal_link, child right_thumb_distal_link, origin xyz=0 0.052 0 rpy=0 0 0, axis 1 0 0, limit lower=0 upper=1.0472 effort=1.1 velocity=2.5303, mimic joint=right_thumb_proximal_joint multiplier=1 offset=0
- added joint right_thumb_metacarpal_joint: type revolute, parent right_base_link, child right_thumb_metacarpal_link, origin xyz=0.005619 0.019867 0.027825 rpy=3.1416 0 2.9637, axis 0 0 1, limit lower=0 upper=1.5184 effort=0.5 velocity=2.6175
- added joint right_thumb_proximal_joint: type revolute, parent right_thumb_metacarpal_link, child right_thumb_proximal_link, origin xyz=0 0.014227 0 rpy=-2.9667 -0.23736 2.9737, axis 1 0 0, limit lower=0 upper=1.0472 effort=1.1 velocity=2.5303
- added joint right_thumb_tip: type fixed, parent right_thumb_distal_link, child right_thumb_tip, origin xyz=0 0.026529 -0.0017734 rpy=-0.06675 -0 0
- joint left_hip_pitch_joint: limit lower=-2.5307 upper=2.8798 effort=88 velocity=32 -> lower=-2.5307 upper=2.8798 effort=139 velocity=20
- joint right_hip_pitch_joint: limit lower=-2.5307 upper=2.8798 effort=88 velocity=32 -> lower=-2.5307 upper=2.8798 effort=139 velocity=20

Commit message: Joints: the G1's original geometry, compressed, instead of decimated STL
Every mesh was decimated to 2000 faces (6.9 MB of STL). Decimation drops
geometry mesh by mesh, so the robot came out lumpy and not even symmetric
(the two sides of the pelvis differed). Now the build keeps all 627k faces
of Unitree's meshes, bakes creased normals (35 degrees) and packs each one
as a meshopt-compressed GLB with gltfpack: 3.1 MB, less than half of
before. The viewer loads them with GLTFLoader + three's MeshoptDecoder
(bundled, no network) and computes no normals of its own.

File: public/g1/g1.urdf (robot description, URDF)
Before this commit: robot g1_29dof_mode_15_brainco_hand, 72 links, 71 joints
Links:
- link head_link: geometry visual mesh filename=meshes/head_link.glb
- link left_ankle_pitch_link: geometry visual mesh filename=meshes/left_ankle_pitch_link.glb
- link left_ankle_roll_link: geometry visual mesh filename=meshes/left_ankle_roll_link.glb
- link left_base2_link: geometry visual mesh filename=meshes/left_base2_link.glb
- link left_base_link: geometry visual mesh filename=meshes/left_base_link.glb
- link left_elbow_link: geometry visual mesh filename=meshes/left_elbow_link.glb
- link left_hip_pitch_link: geometry visual mesh filename=meshes/left_hip_pitch_link.glb
- link left_hip_roll_link: geometry visual mesh filename=meshes/left_hip_roll_link.glb
- link left_hip_yaw_link: geometry visual mesh filename=meshes/left_hip_yaw_link.glb
- link left_index_distal_Link: geometry visual mesh filename=meshes/left_index_distal_Link.glb
- link left_index_proximal_Link: geometry visual mesh filename=meshes/left_index_proximal_Link.glb
- link left_index_tip_Link: geometry visual mesh filename=meshes/left_index_tip_Link.glb
- link left_knee_link: geometry visual mesh filename=meshes/left_knee_link.glb
- link left_middle_distal_Link: geometry visual mesh filename=meshes/left_middle_distal_Link.glb
- link left_middle_proximal_Link: geometry visual mesh filename=meshes/left_middle_proximal_Link.glb
- link left_middle_tip_Link: geometry visual mesh filename=meshes/left_middle_tip_Link.glb
- link left_pinky_distal_Link: geometry visual mesh filename=meshes/left_pinky_distal_Link.glb
- link left_pinky_proximal_Link: geometry visual mesh filename=meshes/left_pinky_proximal_Link.glb
- link left_pinky_tip_Link: geometry visual mesh filename=meshes/left_pinky_tip_Link.glb
- link left_ring_distal_Link: geometry visual mesh filename=meshes/left_ring_distal_Link.glb
- link left_ring_proximal_Link: geometry visual mesh filename=meshes/left_ring_proximal_Link.glb
- link left_ring_tip_Link: geometry visual mesh filename=meshes/left_ring_tip_Link.glb
- link left_shoulder_pitch_link: geometry visual mesh filename=meshes/left_shoulder_pitch_link.glb
- link left_shoulder_roll_link: geometry visual mesh filename=meshes/left_shoulder_roll_link.glb
- link left_shoulder_yaw_link: geometry visual mesh filename=meshes/left_shoulder_yaw_link.glb
- link left_thumb_distal_Link: geometry visual mesh filename=meshes/left_thumb_distal_Link.glb
- link left_thumb_metacarpal_Link: geometry visual mesh filename=meshes/left_thumb_metacarpal_Link.glb
- link left_thumb_proximal_Link: geometry visual mesh filename=meshes/left_thumb_proximal_Link.glb
- link left_thumb_tip_Link: geometry visual mesh filename=meshes/left_thumb_tip_Link.glb
- link left_wrist_pitch_link: geometry visual mesh filename=meshes/left_wrist_pitch_link.glb
- link left_wrist_roll_link: geometry visual mesh filename=meshes/left_wrist_roll_link.glb
- link left_wrist_yaw_link: geometry visual mesh filename=meshes/left_wrist_yaw_link.glb
- link logo_link: geometry visual mesh filename=meshes/logo_link.glb
- link pelvis: geometry visual mesh filename=meshes/pelvis_ver0529.glb
- link right_ankle_pitch_link: geometry visual mesh filename=meshes/right_ankle_pitch_link.glb
- link right_ankle_roll_link: geometry visual mesh filename=meshes/right_ankle_roll_link.glb
- link right_base2_link: geometry visual mesh filename=meshes/right_base2_link.glb
- link right_base_link: geometry visual mesh filename=meshes/right_base_link.glb
- link right_elbow_link: geometry visual mesh filename=meshes/right_elbow_link.glb
- link right_hip_pitch_link: geometry visual mesh filename=meshes/right_hip_pitch_link.glb
- link right_hip_roll_link: geometry visual mesh filename=meshes/right_hip_roll_link.glb
- link right_hip_yaw_link: geometry visual mesh filename=meshes/right_hip_yaw_link.glb
- link right_index_distal_link: geometry visual mesh filename=meshes/right_index_distal_link.glb
- link right_index_proximal_link: geometry visual mesh filename=meshes/right_index_proximal_link.glb
- link right_index_tip: geometry visual mesh filename=meshes/right_index_tip.glb
- link right_knee_link: geometry visual mesh filename=meshes/right_knee_link.glb
- link right_middle_distal_link: geometry visual mesh filename=meshes/right_middle_distal_link.glb
- link right_middle_proximal_link: geometry visual mesh filename=meshes/right_middle_proximal_link.glb
- link right_middle_tip: geometry visual mesh filename=meshes/right_middle_tip.glb
- link right_pinky_distal_link: geometry visual mesh filename=meshes/right_pinky_distal_link.glb
- link right_pinky_proximal_link: geometry visual mesh filename=meshes/right_pinky_proximal_link.glb
- link right_pinky_tip: geometry visual mesh filename=meshes/right_pinky_tip.glb
- link right_ring_distal_link: geometry visual mesh filename=meshes/right_ring_distal_link.glb
- link right_ring_proximal_link: geometry visual mesh filename=meshes/right_ring_proximal_link.glb
- link right_ring_tip: geometry visual mesh filename=meshes/right_ring_tip.glb
- link right_shoulder_pitch_link: geometry visual mesh filename=meshes/right_shoulder_pitch_link.glb
- link right_shoulder_roll_link: geometry visual mesh filename=meshes/right_shoulder_roll_link.glb
- link right_shoulder_yaw_link: geometry visual mesh filename=meshes/right_shoulder_yaw_link.glb
- link right_thumb_distal_link: geometry visual mesh filename=meshes/right_thumb_distal_link.glb
- link right_thumb_metacarpal_link: geometry visual mesh filename=meshes/right_thumb_metacarpal_link.glb
- link right_thumb_proximal_link: geometry visual mesh filename=meshes/right_thumb_proximal_link.glb
- link right_thumb_tip: geometry visual mesh filename=meshes/right_thumb_tip.glb
- link right_wrist_pitch_link: geometry visual mesh filename=meshes/right_wrist_pitch_link.glb
- link right_wrist_roll_link: geometry visual mesh filename=meshes/right_wrist_roll_link.glb
- link right_wrist_yaw_link: geometry visual mesh filename=meshes/right_wrist_yaw_link.glb
- link torso_link: geometry visual mesh filename=meshes/torso_link_rev_1_0.glb
- link waist_roll_link: geometry visual mesh filename=meshes/waist_roll_link_rev_1_0.glb
- link waist_yaw_link: geometry visual mesh filename=meshes/waist_yaw_link_rev_1_0.glb

Commit message: Joints: no maker lettering on the chest
The build drops the visual of logo_link (the raised UNITREE letters); the
link and its joint stay so the tree is still Unitree's.

File: public/g1/g1.urdf (robot description, URDF)
Before this commit: robot g1_29dof_mode_15_brainco_hand, 72 links, 71 joints
Links:
- link logo_link: geometry 
